Commit message: [ADD] Added Z index

File: proyecto/robot_ws/src/robot_description/urdf/robot_rrr_proyecto.urdf (robot description, URDF)
Before this commit: robot robot_rrr_proyecto, 4 links, 3 joints
Links:
- link base_link: geometry visual cylinder length=0.1 radius=0.15; visual cylinder length=0.2 radius=0.05
Joints:
- joint arm_joint: axis 0 0 1 -> 0 1 0
- joint forearm_joint: axis 0 0 1 -> 0 1 0
- joint shoulder_joint: origin xyz=0 0 0.1 rpy=0 0 0 -> xyz=0 0 0.3 rpy=0 0 0

Commit message: [PROYECTO] Cinemática inversa robusta y yaw 360° para brazo RRR

File: proyecto/robot_ws/src/robot_description/urdf/robot_rrr_proyecto.urdf (robot description, URDF)
Before this commit: robot robot_rrr_proyecto, 4 links, 3 joints
Joints:
- joint shoulder_joint: limit lower=-3.14 upper=3.14 effort=10.0 velocity=10.0 -> effort=10.0 velocity=10.0; type revolute -> continuous
